File: MCF8316A1VRGFR/MCF8316A1VRGFR.kicad_sch (KiCad schematic)
At the start: 18 parts, among them IC1 MCF8316A1VRGFR, M1 BLDC Motor, U1 ESP32-S3-DevKitC

Commit message: mcf code
Parts:
- added R8: 10k, symbol Device:R
Connections:
- net +3V3: now also R8.2
- net DIR: now also R8.1
Other:
- moved on the sheet: R1
Changed lines of the file:
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@@
   (junction (at 146.05 102.87) (diameter 0) (color 0 0 0 0)
   )
-  (junction (at 248.92 83.82) (diameter 0) (color 0 0 0 0)
-  )
   (junction (at 185.42 114.3) (diameter 0) (color 0 0 0 0)
   )
@@
   )
   (junction (at 223.52 134.62) (diameter 0) (color 0 0 0 0)
+  )
+  (junction (at 251.46 80.01) (diameter 0) (color 0 0 0 0)
+  )
+  (junction (at 248.92 88.265) (diameter 0) (color 0 0 0 0)
   )
   (junction (at 204.47 102.87) (diameter 0) (color 0 0 0 0)
@@
     (stroke (width 0) (type default))
   )
-  (wire (pts (xy 269.24 83.82) (xy 269.24 87.63))
+  (wire (pts (xy 269.24 88.265) (xy 269.24 92.075))
+    (stroke (width 0) (type default))
+  )
+  (wire (pts (xy 269.24 80.01) (xy 265.43 80.01))
     (stroke (width 0) (type default))
   )
@@
     (stroke (width 0) (type default))
   )
-  (wire (pts (xy 265.43 83.82) (xy 269.24 83.82))
+  (wire (pts (xy 265.43 88.265) (xy 269.24 88.265))
     (stroke (width 0) (type default))
   )
@@
     (stroke (width 0) (type default))
   )
+  (wire (pts (xy 248.92 88.265) (xy 248.92 91.44))
+    (stroke (width 0) (type default))
+  )
   (wire (pts (xy 212.09 149.86) (xy 220.98 149.86))
     (stroke (width 0) (type default))
@@
     (stroke (width 0) (type default))
   )
-  (wire (pts (xy 248.92 83.82) (xy 257.81 83.82))
+  (wire (pts (xy 248.92 88.265) (xy 257.81 88.265))
     (stroke (width 0) (type default))
   )
@@
     (stroke (width 0) (type default))
   )
+  (wire (pts (xy 269.24 73.66) (xy 269.24 80.01))
+    (stroke (width 0) (type default))
+  )
   (wire (pts (xy 199.39 149.86) (xy 212.09 149.86))
     (stroke (width 0) (type default))
@@
     (stroke (width 0) (type default))
   )
-  (wire (pts (xy 251.46 72.39) (xy 251.46 91.44))
+  (wire (pts (xy 251.46 72.39) (xy 251.46 80.01))
     (stroke (width 0) (type default))
   )
@@
     (stroke (width 0) (type default))
   )
+  (wire (pts (xy 251.46 80.01) (xy 251.46 91.44))
+    (stroke (width 0) (type default))
+  )
   (wire (pts (xy 127 102.87) (xy 146.05 102.87))
     (stroke (width 0) (type default))
@@
     (stroke (width 0) (type default))
   )
+  (wire (pts (xy 251.46 80.01) (xy 257.81 80.01))
+    (stroke (width 0) (type default))
+  )
   (wire (pts (xy 204.47 102.87) (xy 204.47 99.06))
     (stroke (width 0) (type default))
@@
     (stroke (width 0) (type default))
   )
-  (wire (pts (xy 248.92 72.39) (xy 248.92 83.82))
-    (stroke (width 0) (type default))
-  )
   (wire (pts (xy 210.82 119.38) (xy 210.82 114.3))
     (stroke (width 0) (type default))
@@
     (stroke (width 0) (type default))
   )
-  (wire (pts (xy 248.92 83.82) (xy 248.92 91.44))
+  (wire (pts (xy 248.92 72.39) (xy 248.92 88.265))
     (stroke (width 0) (type default))
   )
@@
     )
   )
+  (symbol (lib_id "power:+3V3") (at 269.24 73.66 0) (unit 1)
+    (in_bom yes) (on_board yes) (dnp no) (fields_autoplaced)
+    (property "Reference" "#PWR018" (at 269.24 77.47 0)
+      (effects (font (size 1.27 1.27)) hide)
+    )
+    (property "Value" "+3V3" (at 269.24 69.85 0)
+      (effects (font (size 1.27 1.27)))
+    )
+    (property "Footprint" "" (at 269.24 73.66 0)
+      (effects (font (size 1.27 1.27)) hide)
+    )
+    (property "Datasheet" "" (at 269.24 73.66 0)
+      (effects (font (size 1.27 1.27)) hide)
+    )
+    (pin "1")
+    (instances
+      (project "MCF8316A1VRGFR"
+        (path "/4526c1ae-4446-43ca-8990-7fd097c197e5"
+          (reference "#PWR018") (unit 1)
+        )
+      )
+    )
+  )
   (symbol (lib_id "Device:R") (at 146.05 93.98 180) (unit 1)
     (in_bom yes) (on_board yes) (dnp no) (fields_autoplaced)
@@
     )
   )
-  (symbol (lib_id "power:GND") (at 269.24 87.63 0) (unit 1)
-    (in_bom yes) (on_board yes) (dnp no) (fields_autoplaced)
-    (property "Reference" "#PWR010" (at 269.24 93.98 0)
-      (effects (font (size 1.27 1.27)) hide)
-    )
-    (property "Value" "GND" (at 269.24 92.71 0)
-      (effects (font (size 1.27 1.27)))
-    )
-    (property "Footprint" "" (at 269.24 87.63 0)
-      (effects (font (size 1.27 1.27)) hide)
-    )
-    (property "Datasheet" "" (at 269.24 87.63 0)
+  (symbol (lib_id "power:GND") (at 269.24 92.075 0) (unit 1)
+    (in_bom yes) (on_board yes) (dnp no) (fields_autoplaced)
+    (property "Reference" "#PWR010" (at 269.24 98.425 0)
+      (effects (font (size 1.27 1.27)) hide)
+    )
+    (property "Value" "GND" (at 269.24 97.155 0)
+      (effects (font (size 1.27 1.27)))
+    )
+    (property "Footprint" "" (at 269.24 92.075 0)
+      (effects (font (size 1.27 1.27)) hide)
+    )
+    (property "Datasheet" "" (at 269.24 92.075 0)
       (effects (font (size 1.27 1.27)) hide)
     )
@@
     )
   )
-  (symbol (lib_id "Device:R") (at 261.62 83.82 90) (unit 1)
-    (in_bom yes) (on_board yes) (dnp no) (fields_autoplaced)
-    (property "Reference" "R1" (at 261.62 78.74 90)
-      (effects (font (size 1.27 1.27)))
-    )
-    (property "Value" "10k" (at 261.62 81.28 90)
-      (effects (font (size 1.27 1.27)))
-    )
-    (property "Footprint" "" (at 261.62 85.598 90)
-      (effects (font (size 1.27 1.27)) hide)
-    )
-    (property "Datasheet" "~" (at 261.62 83.82 0)
+  (symbol (lib_id "Device:R") (at 261.62 88.265 90) (unit 1)
+    (in_bom yes) (on_board yes) (dnp no) (fields_autoplaced)
+    (property "Reference" "R1" (at 261.62 83.185 90)
+      (effects (font (size 1.27 1.27)))
+    )
+    (property "Value" "10k" (at 261.62 85.725 90)
+      (effects (font (size 1.27 1.27)))
+    )
+    (property "Footprint" "" (at 261.62 90.043 90)
+      (effects (font (size 1.27 1.27)) hide)
+    )
+    (property "Datasheet" "~" (at 261.62 88.265 0)
       (effects (font (size 1.27 1.27)) hide)
     )
@@
         )
       )
+    )
+  )
+  (symbol (lib_id "Device:R") (at 261.62 80.01 90) (unit 1)
+    (in_bom yes) (on_board yes) (dnp no) (fields_autoplaced)
+    (property "Reference" "R8" (at 261.62 74.93 90)
+      (effects (font (size 1.27 1.27)))
+    )
+    (property "Value" "10k" (at 261.62 77.47 90)
+      (effects (font (size 1.27 1.27)))
+    )
+    (property "Footprint" "" (at 261.62 81.788 90)
+      (effects (font (size 1.27 1.27)) hide)
+    )
+    (property "Datasheet" "~" (at 261.62 80.01 0)
+      (effects (font (size 1.27 1.27)) hide)
+    )
+    (pin "1")
+    (pin "2")
+    (instances
+      (project "MCF8316A1VRGFR"
+        (path "/4526c1ae-4446-43ca-8990-7fd097c197e5"
+          (reference "R8") (unit 1)
+        )
+      )
